File: KiCad_UFIIC_Display/UFIIC_Display.kicad_pcb (KiCad board)
At the start: 2 copper layers, 74.2 x 31.5 mm, 37 parts, among them Q1 BC639, Q2 BSS138, Q3 BSS138, Q4 BC547, SW1 SW_Push, U1 AMS1117-3.3, U2 STM32F030F4P6

Commit message: Backlight powered by 5V step up
+ backlight is powered by 5V step-up
+ removed unnecessary KiCad files
+ updated .gitignore
Parts:
- removed R15: 330R, Resistor_SMD:R_1206_3216Metric
- moved G*** 0.36 mm to (178.0, 55.9)
- renumbered SW1 to RESET
Connections:
- HD44780 pad A: Net-(R15-Pad1) -> Net-(Q4-Pad3)
- HD44780 pad D0: Net-(U3-PadD0) -> (no net)
- HD44780 pad D1: Net-(U3-PadD1) -> (no net)
- HD44780 pad D2: Net-(U3-PadD2) -> (no net)
- HD44780 pad D3: Net-(U3-PadD3) -> (no net)
- Q4 pad 1: +3V3 -> /+5V
Routing:
- net Net-(Q4-Pad3): track 4.31 -> 16.0 mm
- net Net-(R15-Pad1): track 8.92 -> 0.00 mm
- net /+5V: track 97.3 -> 105.9 mm
- net +3V3: track 213.3 -> 208.1 mm, vias 7 -> 9
